File: PCB/lighting_keypad/lighting_keypad.kicad_pcb (KiCad board)
At the start: 2 copper layers, 98 x 124 mm, 50 parts, among them J1 Conn_01x06_Pin, J2 Conn_01x03_Pin, M2 RP2040_ZERO, SW16 RotaryEncoder, U1 STP16CP05XT, U2 LM1117MP-3.3

Commit message: Completed Rev.B
Parts:
- removed G1, G2: LOGO, ildus_footprints:OSHWLOGO0.3IN
- removed RP1: raspberry_pi_zero_outline, ildus_footprints:raspberry_pi_zero_outline
- added D1: 1N914WT, Diode_SMD:D_SOD-523, F.Cu at (190.0, 52.0)
- added J3: Conn_02x20_Odd_Even, ildus_footprints:raspberry_pi_zero_outline, F.Cu at (149.0, 44.0)
- added J4: Conn_01x03_Pin, Connector_PinHeader_2.54mm:PinHeader_1x03_P2.54mm_Vertical, B.Cu at (139.4, 61.0)
- added R8: 4.7K, Resistor_SMD:R_0603_1608Metric_Pad0.98x0.95mm_HandSolder, F.Cu at (174.3, 65.3)
- J1: moved to F.Cu
- moved J1 71.0 mm to (186.0, 51.1), turned to 180 degrees
- moved C6 7.98 mm to (114.2, 49.0), turned to -90 degrees
- moved R2 4.62 mm to (157.0, 63.5)
- moved R1 4.61 mm to (160.0, 63.5)
- moved C3 3.91 mm to (109.8, 64.2)
- moved C5 3.91 mm to (115.2, 64.2)
- moved JP1 3.58 mm to (187.2, 57.8), turned to -90 degrees
- moved C1 3.31 mm to (109.8, 74.0)
- moved C2 3.31 mm to (115.2, 74.0)
- moved U1 3.15 mm to (128.2, 70.0)
- moved C4 3.08 mm to (107.8, 54.6), turned to 0 degrees
- moved R3 2.91 mm to (120.0, 65.0), turned to -90 degrees
Connections:
- net /UART_RX renamed /RP2040_RX
- net /UART_TX renamed /RP2040_TX
- J1 pad 6: unconnected-(J1-Pin_6-Pad6) -> +3.3RPI
- JP1 pad 2: +5V -> Net-(D1-K)
- M2 pad 19: unconnected-(M2-GPIO28-Pad19) -> /RREQ
- U1 pad 2: Net-(M2-GPIO14) -> Net-(M2-GPIO15)
- U1 pad 3: Net-(M2-GPIO15) -> Net-(M2-GPIO14)
Routing:
- net /RREQ: track 0.00 -> 73.9 mm, vias 0 -> 2
- net +3.3RPI: track 0.00 -> 68.3 mm
- net /I2C_SDA: track 72.7 -> 101.1 mm, vias 1 -> 4
- net /I2C_SCL: track 76.7 -> 98.0 mm, vias 1 -> 4
- net +3V3_RP2040: track 120.4 -> 137.8 mm, vias 2 -> 3
- net +3.3V: track 48.1 -> 32.9 mm
- net /RPI_TX: track 0.00 -> 13.0 mm, vias 0 -> 2
- net /RPI_RX: track 0.00 -> 12.4 mm, vias 0 -> 1
- net Net-(JP1-A): track 31.5 -> 22.4 mm
- net GND: track 263.5 -> 270.3 mm
- net +5V: track 321.5 -> 327.8 mm
- net Net-(D1-K): track 0.00 -> 5.10 mm
- net Net-(U1-~{OUT9}): track 80.8 -> 84.5 mm
- net Net-(U1-~{OUT0}): track 46.6 -> 42.9 mm
- net Net-(M2-GPIO15): track 55.6 -> 58.9 mm
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Other:
- board text added: "Lighting Keypad Rev.B Designed by: IldusV 2 Feb 2026"
- board text removed: "Lighting Keypad Rev.A Design by: IldusV 12 Feb 2025"
