File: PCB/lighting_keypad/lighting_keypad.kicad_sch (KiCad schematic)
At the start: 37 parts, among them J1 Conn_01x06_Pin, J2 Conn_01x03_Pin, M2 RP2040_ZERO, SW16 RotaryEncoder, U1 STP16CP05XT, U2 LM1117MP-3.3

Commit message: Completed Rev.B
Parts:
- added D1: 1N914WT, Diode_SMD:D_SOD-523, symbol Diode:1N914WT
- added J3: Conn_02x20_Odd_Even, ildus_footprints:raspberry_pi_zero_outline, symbol Connector_Generic:Conn_02x20_Odd_Even
- added J4: Conn_01x03_Pin, Connector_PinHeader_2.54mm:PinHeader_1x03_P2.54mm_Vertical, symbol Connector:Conn_01x03_Pin
- added R8: 4.7K, Resistor_SMD:R_0603_1608Metric_Pad0.98x0.95mm_HandSolder, symbol Device:R
Connections:
- net +3V3_RP2040: now also R8.1
- net +5V: now also D1.2 (A), J3.2 (Pin_2), J3.4 (Pin_4); no longer JP1.2 (B)
- net GND: now also J3.14 (Pin_14), J4.1 (Pin_1)
- net I2C_SCL: now also J3.5 (Pin_5)
- net I2C_SDA: now also J3.3 (Pin_3)
- net at U1.2 (SDI): now also M2.16 (GPIO15); no longer M2.15 (GPIO14)
- net at U1.3 (CLK): now also M2.15 (GPIO14); no longer M2.16 (GPIO15)
- net RREQ: now reaches M2.19 (GPIO28)
- net RREQ: now also J3.7 (Pin_7), R8.2
- net +3.3RPI: now reaches J1.6 (Pin_6)
- net +3.3RPI: now also J3.1 (Pin_1)
- net UART_RX renamed RP2040_RX
- net UART_TX renamed RP2040_TX
- new net: D1.1 (K), JP1.2 (B)
- new net RPI_RX: J3.10 (Pin_10), J4.3 (Pin_3)
- new net RPI_TX: J3.8 (Pin_8), J4.2 (Pin_2)
- no-connect marks 36 -> 65
Other:
- note added: "DISPLAY CONTROL INTERFACE"
- note added: "RASPBERRYPI ZERO INTERFACE"
- note added: "REMOVE JUMPER BEFORE PLUGGING USB CABLE"
- note added: "RP2040 UART INTERFACE"
- note added: "RPI UART INTERFACE"
- note removed: "CONTROL INTERFACE"
- note removed: "DEBUG INTERFACE"
- note removed: "REMOVE THE JUMPER BEFORE PLUGGING USB CABLE"
- moved on the sheet: C1, C2, C3, C4, C5, C6, C7, C8, J1, J2, JP1, M2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
